File: kits.sch (KiCad schematic (older format))
At the start: 57 parts, among them J1 10118192-0002LF, J2 S2B-PH-SM4-TB(LF)(SN), Q1 BSS138, Q2 BSS138, SW1 JS202011JCQN, SW2 TL3342F160QG, U1 MCP73811T-420I-OT, U2 TCR2EF18,LM(CT, U3 ATmega32U4RC-MU, U4 ICM-20948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

Commit message: Update kicad version.
Parts:
- U3: symbol MCU_Microchip_ATmega:ATmega32U4RC-MU -> kits-rescue:ATmega32U4RC-MU-MCU_Microchip_ATmega
Changed lines of the file:
@@
 EESchema Schematic File Version 4
-LIBS:kits-cache
-EELAYER 29 0
+EELAYER 30 0
 EELAYER END
 $Descr A4 11693 8268
@@
 Connection ~ 9350 4450
 $Comp
-L MCU_Microchip_ATmega:ATmega32U4RC-MU U3
+L kits-rescue:ATmega32U4RC-MU-MCU_Microchip_ATmega U3
 U 1 1 5D190878
 P 9350 2650
